Commit message: Refactor SVO and BAG pipeline services for improved grasp estimation and video extraction
- Enhanced grasp estimation logic in SVO pipeline to utilize initial object position and smooth distance calculations.
- Updated GMM segmentation in SVO pipeline to align with paper algorithms for release detection.
- Introduced a new generic video extraction service to handle frame, depth, and camera intrinsics extraction from video files.
- Improved video reconstruction methods to prioritize compatibility with various codecs.
- Added error handling and logging for better debugging and user feedback.
- Refined camera intrinsics estimation based on video resolution and common focal length assumptions.

File: data/Common/robot_models/openarm/_sanitized__sanitized_openarm.urdf (robot description, URDF)
Before this commit: robot openarm, 26 links, 25 joints
Links:
- link openarm_body_link0: geometry visual mesh filename=C:/Users/MohammadhoseinAbdoll/I-Genius/data/Common/robot_mo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 scale=0.001 0.001 0.001
- link openarm_left_hand: geometry visual mesh filename=C:/Users/MohammadhoseinAbdoll/I-Genius/data/Common/robot_mo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 scale=0.001 0.001 0.001
- link openarm_left_left_finger: geometry visual mesh filename=C:/Users/MohammadhoseinAbdoll/I-Genius/data/Common/robot_mo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 scale=0.001 0.001 0.001
- link openarm_left_link0: geometry visual mesh filename=C:/Users/MohammadhoseinAbdoll/I-Genius/data/Common/robot_mo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 scale=0.001 -0.001 0.001
- link openarm_left_link1: geometry visual mesh filename=C:/Users/MohammadhoseinAbdoll/I-Genius/data/Common/robot_mo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 scale=0.001 -0.001 0.001
- link openarm_left_link2: geometry visual mesh filename=C:/Users/MohammadhoseinAbdoll/I-Genius/data/Common/robot_mo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 scale=0.001 -0.001 0.001
- link openarm_left_link3: geometry visual mesh filename=C:/Users/MohammadhoseinAbdoll/I-Genius/data/Common/robot_mo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 scale=0.001 -0.001 0.001
- link openarm_left_link4: geometry visual mesh filename=C:/Users/MohammadhoseinAbdoll/I-Genius/data/Common/robot_mo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 scale=0.001 -0.001 0.001
- link openarm_left_link5: geometry visual mesh filename=C:/Users/MohammadhoseinAbdoll/I-Genius/data/Common/robot_mo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 scale=0.001 -0.001 0.001
- link openarm_left_link6: geometry visual mesh filename=C:/Users/MohammadhoseinAbdoll/I-Genius/data/Common/robot_mo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 scale=0.001 -0.001 0.001
- link openarm_left_link7: geometry visual mesh filename=C:/Users/MohammadhoseinAbdoll/I-Genius/data/Common/robot_mo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 scale=0.001 -0.001 0.001
- link openarm_left_right_finger: geometry visual mesh filename=C:/Users/MohammadhoseinAbdoll/I-Genius/data/Common/robot_mo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 scale=0.001 -0.001 0.001
- link openarm_right_hand: geometry visual mesh filename=C:/Users/MohammadhoseinAbdoll/I-Genius/data/Common/robot_mo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 scale=0.001 0.001 0.001
- link openarm_right_left_finger: geometry visual mesh filename=C:/Users/MohammadhoseinAbdoll/I-Genius/data/Common/robot_mo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 scale=0.001 0.001 0.001
- link openarm_right_link0: geometry visual mesh filename=C:/Users/MohammadhoseinAbdoll/I-Genius/data/Common/robot_mo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 scale=0.001 0.001 0.001
- link openarm_right_link1: geometry visual mesh filename=C:/Users/MohammadhoseinAbdoll/I-Genius/data/Common/robot_mo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 scale=0.001 0.001 0.001
- link openarm_right_link2: geometry visual mesh filename=C:/Users/MohammadhoseinAbdoll/I-Genius/data/Common/robot_mo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 scale=0.001 0.001 0.001
- link openarm_right_link3: geometry visual mesh filename=C:/Users/MohammadhoseinAbdoll/I-Genius/data/Common/robot_mo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 scale=0.001 0.001 0.001
- link openarm_right_link4: geometry visual mesh filename=C:/Users/MohammadhoseinAbdoll/I-Genius/data/Common/robot_mo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 scale=0.001 0.001 0.001
- link openarm_right_link5: geometry visual mesh filename=C:/Users/MohammadhoseinAbdoll/I-Genius/data/Common/robot_mo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 scale=0.001 0.001 0.001
- link openarm_right_link6: geometry visual mesh filename=C:/Users/MohammadhoseinAbdoll/I-Genius/data/Common/robot_mo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 scale=0.001 0.001 0.001
- link openarm_right_link7: geometry visual mesh filename=C:/Users/MohammadhoseinAbdoll/I-Genius/data/Common/robot_mo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 scale=0.001 0.001 0.001
- link openarm_right_right_finger: geometry visual mesh filename=C:/Users/MohammadhoseinAbdoll/I-Genius/data/Common/robot_mo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 scale=0.001 -0.001 0.001
